File: MoodLogger_v1/MoodLogger_v1.kicad_pcb (KiCad board)
At the start: 2 copper layers, 46 parts, among them J2 USB_C_Receptacle, Q1 DMG3415U, SW2 SW_MEC_5E, SW3 SW_MEC_5E, SW4 Slide_Switch_SPDT, SW5 SW_MEC_5E, SW6 SW_MEC_5E, U1 ATSAMD21G18A-A, U2 RV-3028-C7, U5 AP2112K-3.3TRG1, U6 MCP73831T-2ACI/OT, U7 W25Q32JVSS, Y1 32.768kHz

Commit message: updated schematic and pcb
Parts:
- removed C2, C3, C5: 100nF, PCM_JLCPCB:C_0402
- removed C4: 1uF, PCM_JLCPCB:C_0402
- removed R4, R5: 10kΩ, PCM_JLCPCB:R_0402
- added C21: 10µF, Capacitor_SMD:C_0805_2012Metric_Pad1.18x1.45mm_HandSolder, F.Cu at (187.2, 60.4)
- added C22: 22pF, Capacitor_SMD:C_0402_1005Metric_Pad0.74x0.62mm_HandSolder, F.Cu at (158.2, 60.9)
- added C23: 22pF, Capacitor_SMD:C_0402_1005Metric_Pad0.74x0.62mm_HandSolder, F.Cu at (157.5, 60.2)
- added CHG2: ORANGE, LED_SMD:LED_0402_1005Metric_Pad0.77x0.64mm_HandSolder, F.Cu at (185.2, 53.8)
- added D2: MBR120, Diode_SMD:D_SOD-123, F.Cu at (175.9, 43.8)
- added J3: JST_2mm_LiPo, PCM_SparkFun-Connector:JST_1x02_P2.0mm_Horizontal_SMD, F.Cu at (193.8, 48.2)
- added R14: 1K, PCM_Resistor_SMD_AKL:R_0402_1005Metric_Pad0.72x0.64mm_HandSolder, F.Cu at (185.2, 55.1)
- added R15: 10K\, PCM_Resistor_SMD_AKL:R_0402_1005Metric_Pad0.72x0.64mm_HandSolder, F.Cu at (188.0, 55.1)
- C1, C18, C6: footprint PCM_JLCPCB:C_0402 -> Capacitor_SMD:C_0402_1005Metric_Pad0.74x0.62mm_HandSolder
- C10, C15, C16, C17: footprint Capacitor_SMD:C_0603_1608Metric -> Capacitor_SMD:C_0402_1005Metric_Pad0.74x0.62mm_HandSolder
- C19, C20: footprint PCM_JLCPCB:C_0603 -> Capacitor_SMD:C_0805_2012Metric_Pad1.18x1.45mm_HandSolder
- R1, R2: footprint PCM_Resistor_SMD_AKL:R_0603_1608Metric -> PCM_Resistor_SMD_AKL:R_0402_1005Metric_Pad0.72x0.64mm_HandSolder
- R10, R11, R12, R19, R20, R21, R9: footprint Resistor_SMD:R_0603_1608Metric -> PCM_Resistor_SMD_AKL:R_0402_1005Metric_Pad0.72x0.64mm_HandSolder
- R16, R17, R18, R22, R23, R6, R7: footprint PCM_JLCPCB:R_0402 -> PCM_Resistor_SMD_AKL:R_0402_1005Metric_Pad0.72x0.64mm_HandSolder
- SW2, SW3, SW5, SW6: footprint Button_Switch_SMD:SW_Push_1P1T_NO_CK_PTS125Sx43PSMTR -> PCM_SparkFun-Switch:Push_SMD_5.2x5.2mm_h2.5mm
- moved U5 70.7 mm to (180.6, 42.9)
- moved C6 64.6 mm to (209.6, 77.8), turned to 180 degrees
- moved C19 64.5 mm to (180.7, 40.0)
- moved R7 61.8 mm to (209.6, 76.0)
- moved R6 61.8 mm to (209.6, 74.1)
- moved U7 59.9 mm to (184.2, 77.2), turned to -90 degrees
- moved R13 59.4 mm to (184.0, 44.5)
- moved Q1 58.8 mm to (176.6, 40.7), turned to 90 degrees
- moved C20 58.4 mm to (176.1, 46.8), turned to -90 degrees
- moved U6 57.1 mm to (187.2, 57.6)
- moved U2 54.7 mm to (206.7, 76.5)
- moved C18 53.1 mm to (184.0, 43.3)
- moved R17 48.2 mm to (192.8, 59.2)
- moved R16 47.9 mm to (192.8, 57.9)
- moved R18 47.1 mm to (173.8, 45.5)
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Connections:
- Y1 pad 1: Net-(U1-PA01) -> unconnected-(Y1-Pad1)
- Y1 pad 2: Net-(U1-PA00) -> unconnected-(Y1-Pad2)
Routing:
- net /5V_TO_SWITCH: track 0.00 -> 2.64 mm
- net Net-(J2-CC2): track 0.00 -> 2.06 mm
- net GND: track 0.00 -> 1.91 mm
Other:
- board outline added: 30 x 30 mm
