File: MoodLogger_v1/MoodLogger_v1.kicad_sch (KiCad schematic)
At the start: 70 parts, among them J1 Conn_01x02_Socket, J2 USB_C_Receptacle, Q1 DMG3415U, SW1 SW_Push, SW2 SW_MEC_5E, SW3 SW_MEC_5E, SW4 Slide_Switch_SPDT, SW5 SW_MEC_5E, SW6 SW_MEC_5E, U1 ATSAMD21G18A-A, U2 RV-3028-C7, U3 SPX3819-3.3, U5 AP2112K-3.3TRG1, U6 MCP73831T-2ACI/OT, U7 W25Q32JVSS, X1 JSTPH, Y1 32.768kHz

Commit message: updated schematic and pcb
Parts:
- removed C2, C3, C5: 100nF, PCM_JLCPCB:C_0402, symbol PCM_JLCPCB-Capacitors:0402,100nF
- removed C4: 1uF, PCM_JLCPCB:C_0402, symbol PCM_JLCPCB-Capacitors:0402,1uF
- removed R4, R5: 10kΩ, PCM_JLCPCB:R_0402, symbol PCM_JLCPCB-Resistors:0402,10kΩ
- added J3: JST_2mm_LiPo, PCM_SparkFun-Connector:JST_1x02_P2.0mm_Horizontal_SMD, symbol PCM_SparkFun-Connector:Conn_01x02_JST_P2.0mm_Horizontal_SMD
- C1, C18, C6: footprint PCM_JLCPCB:C_0402 -> Capacitor_SMD:C_0402_1005Metric_Pad0.74x0.62mm_HandSolder
- C10, C15, C16, C17: footprint Capacitor_SMD:C_0603_1608Metric -> Capacitor_SMD:C_0402_1005Metric_Pad0.74x0.62mm_HandSolder
- C19, C20: footprint PCM_JLCPCB:C_0603 -> Capacitor_SMD:C_0805_2012Metric_Pad1.18x1.45mm_HandSolder
- C21: footprint Adafruit Feather M0 Basic rev C:0805-NO -> Capacitor_SMD:C_0805_2012Metric_Pad1.18x1.45mm_HandSolder
- C22, C23: footprint Adafruit Feather M0 Basic rev C:0603-NO -> Capacitor_SMD:C_0402_1005Metric_Pad0.74x0.62mm_HandSolder
- CHG2: footprint Adafruit Feather M0 Basic rev C:CHIPLED_0805_NOOUTLINE -> LED_SMD:LED_0402_1005Metric_Pad0.77x0.64mm_HandSolder
- D2: footprint Adafruit Feather M0 Basic rev C:SOD-123 -> Diode_SMD:D_SOD-123
- R1, R2: footprint PCM_Resistor_SMD_AKL:R_0603_1608Metric -> PCM_Resistor_SMD_AKL:R_0402_1005Metric_Pad0.72x0.64mm_HandSolder
- R10, R11, R12, R19, R20, R21, R9: footprint Resistor_SMD:R_0603_1608Metric -> PCM_Resistor_SMD_AKL:R_0402_1005Metric_Pad0.72x0.64mm_HandSolder
- R14, R15: footprint Adafruit Feather M0 Basic rev C:0603-NO -> PCM_Resistor_SMD_AKL:R_0402_1005Metric_Pad0.72x0.64mm_HandSolder
- R16, R17, R18, R22, R23, R6, R7: footprint PCM_JLCPCB:R_0402 -> PCM_Resistor_SMD_AKL:R_0402_1005Metric_Pad0.72x0.64mm_HandSolder
- SW2, SW3, SW5, SW6: footprint Button_Switch_SMD:SW_Push_1P1T_NO_CK_PTS125Sx43PSMTR -> PCM_SparkFun-Switch:Push_SMD_5.2x5.2mm_h2.5mm
Connections:
- net GND: now also J3.1 (-)
- net VBATT: now also J3.2 (+)
- net VBUS: now also D2.2 (A); no longer D2.A
- net at C20.1, Q1.2 (S), R13.1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: now also D2.1 (C); no longer D2.C
- net at C22.1, U1.2 (PA01): no longer Y1.1
- net at C23.1, U1.1 (PA00): no longer Y1.2
Other:
- note added: "Battery Connector"
- moved on the sheet: R18, Y1
